File: Design/P08R6.sch (EAGLE design)
At the start: 28 parts, among them P1 PENTABIT_17.32, U1 STM32F091CBU6, U2 VL53L0X, X1 XTALL_CSTCE8M00G52

Commit message: no message
Parts:
- removed B, C, D: PAD1, Hexabitz:PAD1
- removed C3: 100nF, Hexabitz:C-0603
- removed C4: 4.7uF, Hexabitz:C-0805-POL
- added C12: 10uF, HEXABITZ_RCLS:C-0402
- added C13: 1uF, HEXABITZ_RCLS:C-0402
- added C14, C15, C16, C17: 100nF, HEXABITZ_RCLS:C-0402
- added D2: BOURNS_CDSOD323-T03SCBOURNS_CDSOD323-T03SC_0_0, HEXABITZ_RCLS:BOURNS_CDSOD323-T03SCBOURNS_CDSOD323-T03SC_0_0
- added JP2: (no value), pinhead:PINHD-1X3
- added R10, R8, R9: 47k, HEXABITZ_RCLS:R-0402
- added R11: 10k, HEXABITZ_RCLS:R-0402
- added R12: 100k, HEXABITZ_RCLS:R-0402
- added TRIMBLE-LOGO1: HEXA-LOGO, HEXABITZ_USER_INTERFACE_PARTS:HEXA-LOGO
- added U3: LDK130PU18R, HEXABITZ_ICs:LDK130PU18R
- added U4: TCK107AG,LF, HEXABITZ_ICs:TCK107AG,LF
- added U5, U6: PI4ULS3V204ZBEX, HEXABITZ_ICs:PI4ULS3V204ZBEX
- C1: value 10nF -> 100nF; device Hexabitz:C-0603 -> HEXABITZ_RCLS:C-0402; CAPACITANCE 10nF -> (none); MFN KEMET -> (none); MPN C0603C103K5RACTU -> (none); OCTOPART_URL https://octopart.com/c0603c103k5ractu-kemet-133094?r=sp&s=R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 -> (none); TOLERANCE 10% -> (none); VOLTAGE_RATING 50V -> (none)
- C10: device Hexabitz:C-0603 -> HEXABITZ_RCLS:C-0402; CAPACITANCE 100 nF -> (none); MFN KEMET -> (none); MPN C0603C104K8RACTU -> (none); OCTOPART_URL https://octopart.com/0603yc104k4t2a-avx+interconnect+%2F+el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 -> (none); TOLERANCE ±10% -> (none); VOLTAGE_RATING 16.0 V -> (none)
- C11: device Hexabitz:C-0805 -> HEXABITZ_RCLS:C-0603; CAPACITANCE 4.7µF -> (none); MFN Murata -> (none); MPN GRM21BC81E475KA12L -> (none); OCTOPART_URL https://octopart.com/grm21bc81e475ka12l-murata-10331911?r=s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 -> (none); TOLERANCE 10% -> (none); VOLTAGE_RATING 25V -> (none)
- C2: value 1.00uF -> 1uF; device Hexabitz:C-0805-POL -> HEXABITZ_RCLS:C-0603-POL; CAPACITANCE 1.00uF -> (none); MFN Yageo -> (none); MPN CC0805KKX7R7BB105 -> (none); OCTOPART_URL https://octopart.com/cc0805kkx7r7bb105-yageo-8376555?r=sp&s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 -> (none); TOLERANCE 10% -> (none); VOLTAGE_RATING 16V -> (none)
- C5: device Hexabitz:C-0603 -> HEXABITZ_RCLS:C-0402; CAPACITANCE 100nF -> (none); MFN KEMET -> (none); MPN C0603C104K8RACTU -> (none); OCTOPART_URL https://octopart.com/c0603c104k8ractu-kemet-145075?r=sp&s=9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 -> (none); TOLERANCE 10% -> (none); VOLTAGE_RATING 10 -> (none)
- C6, C8: device Hexabitz:C-0603 -> HEXABITZ_RCLS:C-0402; CAPACITANCE 100nF -> (none); MFN KEMET -> (none); MPN C0603C104K8RACTU -> (none); OCTOPART_URL https://octopart.com/c0603c104k8ractu-kemet-145075?r=sp&s=9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 -> (none); TOLERANCE 10% -> (none); VOLTAGE_RATING 10V -> (none)
- C7: device Hexabitz:C-0805-POL -> HEXABITZ_RCLS:C-0603-POL; CAPACITANCE 4.7uF -> (none); MFN Murata -> (none); MPN GRM21BC81E475KA12L -> (none); OCTOPART_URL https://octopart.com/grm21bc81e475ka12l-murata-10331911?r=s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 -> (none); TOLERANCE 10% -> (none); VOLTAGE_RATING 25V -> (none)
- C9: device Hexabitz:C-0603 -> HEXABITZ_RCLS:C-0402; CAPACITANCE 100nF -> (none); MFN KEMET -> (none); MPN C0603C104K8RACTU -> (none); OCTOPART_URL https://octopart.com/c0603c104k8ractu-kemet-145075?r=sp&s=9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 -> (none); TOLERANCE 10V -> (none); VOLTAGE_RATING 10% -> (none)
- D1: value VLMS1300-GS08 -> RED; device Hexabitz:VLMS1300-GS08 -> HEXABITZ_USER_INTERFACE_PARTS:VLMS1300-GS08
- FB1: device Hexabitz:FB-TDK_MMZ1608Y300B -> HEXABITZ_RCLS:FB-0603
- R: value PAD1 -> R; device Hexabitz:PAD1 -> HEXABITZ_USER_INTERFACE_PARTS:PINHD-1X1
- R1: value 270.0R -> 270R; device Hexabitz:R-0603 -> HEXABITZ_RCLS:R-0402; MFN Yageo -> (none); MPN RC0603FR-07270RL -> (none); OCTOPART_URL https://octopart.com/search?q=RC0603FR-07270RL&start=0 -> (none); RESISTANCE 270.0 Ohm -> (none); TOLERANCE 1% -> (none)
- R2: device Hexabitz:R-0603 -> HEXABITZ_RCLS:R-0402
- R3: value 10.0K -> 10K; device Hexabitz:R-0603 -> HEXABITZ_RCLS:R-0402; MFN Yageo -> (none); MPN RC0603JR-0710KL -> (none); OCTOPART_URL https://octopart.com/search?q=RC0603JR-0710KL&start=0 -> (none); RESISTANCE 10.0K Ohm -> (none); TOLERANCE 5% -> (none)
- R4: value 2.2k -> 10k; device Hexabitz:R-0603 -> HEXABITZ_RCLS:R-0402; MFN Vishay -> (none); MPN CRCW06032K20FKEA -> (none); OCTOPART_URL https://octopart.com/crcw06032k20fkea-vishay-40018987 -> (none); RESISTANCE 2.2 kΩ -> (none); TOLERANCE ±1% -> (none)
- R5, R6, R7: value 2.2k -> 47k; device Hexabitz:R-0603 -> HEXABITZ_RCLS:R-0402; MFN Vishay -> (none); MPN CRCW06032K20FKEA -> (none); OCTOPART_URL https://octopart.com/crcw06032k20fkea-vishay-40018987 -> (none); RESISTANCE 2.2 kΩ -> (none); TOLERANCE ±1% -> (none)
- U1: value STM32F091CBU6 -> STM32G0B1CEU6QFN_B1CEU6_STM-L; device Hexabitz:STM32F091CBU6 -> HEXABITZ_ICs:STM32G0B1CEU6QFN_B1CEU6_STM-L
- U2: value VL53L0X -> VL53L8CXV0GC_1; device Hexabitz:VL53L0X -> HEXABITZ_ICs:VL53L8CXV0GC_1
- X1: device Hexabitz:XTALL_CSTCE8M00G52 -> HEXABITZ_RCLS:XTALL_CSTCE8M00G52
Connections:
- net UART2_RX renamed USART2_RX
- net UART2_TX renamed USART2_TX
- removed net B1: B.P$1, R3.2, U1.PF11-OSC_BOOT0
- removed net I2C2_SCL: R5.1, U1.PB13, U2.SCL
- removed net I2C2_SDA: R6.1, U1.PB14, U2.SDA
- removed net N$9: C.P$1, U1.PA14
- removed net R1: C8.1, R.P$1, U1.NRST
- removed net UART1_RX: P1.SD5, U1.PA10
- removed net UART1_TX: P1.SU5, U1.PA9
- removed net UART3_RX: P1.SD4, U1.PB11
- removed net UART3_TX: P1.SU4, U1.PB10
- removed net UART4_RX: U1.PA1
- removed net UART4_TX: U1.PA0
- removed net UART5_RX: P1.SD1, U1.PB4
- removed net UART5_TX: P1.SU1, U1.PB3
- removed net UART6_RX: P1.SD3, U1.PA5
- removed net UART6_TX: P1.SU3, U1.PA4
- removed net XSHUT: R4.1, U1.PB0, U2.!XSHUT
- new net +1.8V: C12.1, C15.1, C16.1, C17.1, C9.1, R4.2, R5.2, R6.2, R7.2, R8.2, R9.2, U2.CORE_1V8, U2.IOVDD, U3.OUT, U5.VCCA, U6.VCCB
- new net 1.8V_EN: R12.2, U1.PB5, U3.EN
- new net AVDD_EN: U1.PA11_[PA9], U4.CONTROL
- new net CLK: JP2.1, JP2.2, R3.2, U1.PA14-BOOT0
- new net CONTROLLED_AVDD: C10.1, U2.AVDD, U4.VOUT
- new net DATA: JP2.3, U1.PA13
- new net LPN: U1.PA12_[PA10], U6.A4
- new net MCU_SPI2_MISO: U1.PB6, U5.B1
- new net MCU_SPI2_MOSI: U1.PB7, U5.B2
- new net MCU_SPI2_NSS: U1.PB9, U5.B4
- new net MCU_SPI2_SCK: U1.PB8, U5.B3
- new net N$1: R4.1, U5.EN
- new net N$2: R11.1, U6.EN
- new net SENSOR_INT: R9.1, U2.INT, U6.B1
- new net SENSOR_LPN: R7.1, U2.LPN, U6.B4
- new net SENSOR_MISO: R10.2, U2.MISO, U5.A1
- new net SENSOR_NSS: R5.1, U2.NCS, U5.A4
- new net SENSOR_SCL/MCLK: U2.SCL/MCLK, U5.A3
- new net SENSOR_SDA/MOSI: U2.SDA/MOSI, U5.A2
- new net SENSOR_SPI_I2C_N: R6.1, U2.SPI_I2C_N, U6.B3
- new net SENSOR_SYNC: R8.1, U2.SYNC, U6.B2
- new net SPI_I2C_N: U1.PA15, U6.A3
- new net SYNC: U1.PD0, U6.A2
- new net USART1_RX: P1.SD4, U1.PA10
- new net USART1_TX: P1.SU4, U1.PA9
- new net USART3_RX: P1.SD3, U1.PB11
- new net USART3_TX: P1.SU3, U1.PB10
- new net USART4_RX: P1.SD1, U1.PA1
- new net USART4_TX: P1.SU1, U1.PA0
- new net USART5_RX: P1.SD5, U1.PD2
- new net USART5_TX: P1.SU5, U1.PD3
- net GND: now also C1.2, C11.2, C12.2, C13.2, C14.2, C15.2, C16.2, C17.2, D2.C, R10.1, R12.1, U1.VSS, U2.GND_1, U2.GND_3, U2.RSDV1, U2.RSDV2, U2.RSVD3, U2.THERMALPAD, U3.GND, U4.GND, U5.GND, U6.GND; no longer C11.-, C3.2, C4.-, C5.2, C6.2, C7.-, U1.EP, U1.PA12, U1.PA6, U1.PA7, U1.PB5, U1.PB6, U1.PB7, U1.VSS_0, U1.VSS_1, U1.VSS_2, U2.AVSSVCSEL, U2.GND
- net INT: now also U1.PD1, U6.A1; no longer R7.1, U1.PB2, U2.GPIO1
- net N$3: now also D1.A; no longer U1.PA11
- net N$4: now also C8.1, R.1, U1.PF2-NRST; no longer D1.A, R1.1
- net N$5: now also U1.PF1-OSC_OUT; no longer U1.PF0-OSC_IN
- net N$6: now also U1.PF0-OSC_IN; no longer U1.PF1-OSC_OUT
- net N$7: now also R1.1, U1.PB12; no longer D.P$1, U1.PA13
- net VDD: now also C1.1, C11.1, C13.1, C14.1, D2.A, R11.2, U3.IN, U4.VIN, U5.VCCB, U6.VCCA; no longer C10.1, C11.+, C3.1, C4.+, C5.1, C6.1, C7.+, C9.1, R4.2, R5.2, R6.2, R7.2, U1.VBAT, U1.VDDIO2, U1.VDD_0, U1.VDD_1, U2.AVDD, U2.AVDDVCSEL
- net VDDA: now also C2.1, C5.1, C6.1, C7.1, U1.VBAT, U1.VDD/VDDA, U1.VREF+; no longer C1.1, C2.+, U1.VDDA
- net VSSA: now also C2.2, C5.2, C6.2, C7.2, U1.VSS/VSSA; no longer C1.2, C2.-, U1.VSS_A
Other:
- note added: "1.8V LDO Reguletor"
- note added: "AVDD Controller"
- note added: "Active High"
- note added: "BOOT"
- note added: "Level Shifters"
- note added: "P08R6"
- note added: "P08R6_Backend"
- note added: "P08R6_Frontend"
- note added: "Time-of-Flite sensor"
- note added: "VDD=3.3 Volts"
- note added: "VDD\VDDA Coupling"
- note added: "VL53L8 IR ToF LiDar Sensor"
- note added: "Vref Coupling"
- note removed: "0"
- note removed: "P08R60"
- note removed: "P08R60_Backend"
- note removed: "P08R60_Frontend"
- note removed: "Time-of-Flight IR Sensor"
- note removed: "VBAT"
- note removed: "VDD Coupling"
- note removed: "VDDA Coupling"
- moved on the sheet: C10, C2, C5, C6, C7, C8, D1, FB1, R1, R2, R3, R4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
