File: P08R60/Design/P08R60.sch (EAGLE design)
At the start: 28 parts, among them P1 PENTABIT_17.32, U1 STM32F091CBU6, U2 VL53L0X, X1 XTALL_CSTCE8M00G52

Commit message: Fix R4 to R7 PN
Parts:
- R4, R5, R6, R7: MFN Yageo -> Vishay; MPN RC0603FR-07270RL -> CRCW06032K20FKEA
Changed lines of the file:
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@@
 <part name="SUPPLY17" library="supply2" library_urn="urn:adsk.eagle:library:372" deviceset="VDD" device=""/>
 <part name="R4" library="Hexabitz" deviceset="R-0603" device="" value="2.2k">
-<attribute name="MFN" value="Yageo"/>
-<attribute name="MPN" value="RC0603FR-07270RL"/>
+<attribute name="MFN" value="Vishay"/>
+<attribute name="MPN" value="CRCW06032K20FKEA"/>
 <attribute name="OCTOPART_URL" value="https://octopart.com/crcw06032k20fkea-vishay-40018987"/>
 <attribute name="RESISTANCE" value="2.2 kΩ"/>
@@
 </part>
 <part name="R5" library="Hexabitz" deviceset="R-0603" device="" value="2.2k">
-<attribute name="MFN" value="Yageo"/>
-<attribute name="MPN" value="RC0603FR-07270RL"/>
+<attribute name="MFN" value="Vishay"/>
+<attribute name="MPN" value="CRCW06032K20FKEA"/>
 <attribute name="OCTOPART_URL" value="https://octopart.com/crcw06032k20fkea-vishay-40018987"/>
 <attribute name="RESISTANCE" value="2.2 kΩ"/>
@@
 </part>
 <part name="R6" library="Hexabitz" deviceset="R-0603" device="" value="2.2k">
-<attribute name="MFN" value="Yageo"/>
-<attribute name="MPN" value="RC0603FR-07270RL"/>
+<attribute name="MFN" value="Vishay"/>
+<attribute name="MPN" value="CRCW06032K20FKEA"/>
 <attribute name="OCTOPART_URL" value="https://octopart.com/crcw06032k20fkea-vishay-40018987"/>
 <attribute name="RESISTANCE" value="2.2 kΩ"/>
@@
 <part name="SUPPLY19" library="supply2" library_urn="urn:adsk.eagle:library:372" deviceset="VDD" device=""/>
 <part name="R7" library="Hexabitz" deviceset="R-0603" device="" value="2.2k">
-<attribute name="MFN" value="Yageo"/>
-<attribute name="MPN" value="RC0603FR-07270RL"/>
+<attribute name="MFN" value="Vishay"/>
+<attribute name="MPN" value="CRCW06032K20FKEA"/>
 <attribute name="OCTOPART_URL" value="https://octopart.com/crcw06032k20fkea-vishay-40018987"/>
 <attribute name="RESISTANCE" value="2.2 kΩ"/>
